File: Eagle/GarageDoor.sch (EAGLE design)
At the start: 30 parts, among them Q1 P-FET

Commit message: Changed to positive side sensor control
Parts:
- added Q4, Q5: P-FET, SparkFun-DiscreteSemi:TRANSISTOR_PNPSMD
- added R10, R9: 10K, SparkFun-Resistors:RESISTOR0805-RES
Connections:
- new net N$12: Q2.C, Q5.B, R10.1
- new net N$13: JP3.2, Q5.C
- net +5V: now also Q4.E, Q5.E, R10.2, R9.2; no longer JP2.2, JP3.2
- net GND: now also JP2.1, JP3.1
- net N$2: now also JP2.2, Q4.C; no longer JP2.1, Q3.C
- net N$6: now also Q3.C, Q4.B, R9.1; no longer JP3.1, Q2.C
Other:
- moved on the sheet: ., 3V3, 3V3R, C3, C4, JP1, JP2, JP3, JP4, JP5, JP6, OLED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

Commit message: Changed to NPN output
Parts:
- Q1: value P-FET -> (none); device SparkFun-DiscreteSemi:TRANSISTOR_PNPSMD -> SparkFun-DiscreteSemi:TRANSISTOR_NPNSOT23-3
- R10, R6, R9: value 10K -> 4K7
- R4: value 10K -> 1K
- R5: value 10K -> 5K6
Connections:
- net GND: now also Q1.E; no longer Q1.C
- net N$1: now also Q1.C; no longer Q1.E
Changed lines of the file:
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@@
 <part name="." library="SparkFun-Connectors" deviceset="M02" device="PTH"/>
 <part name="C1" library="SparkFun-Capacitors" deviceset="CAP" device="" value="0.1uF"/>
-<part name="Q1" library="SparkFun-DiscreteSemi" deviceset="TRANSISTOR_PNP" device="SMD" value="P-FET"/>
 <part name="U$3" library="CuriousTech" deviceset="SMD-PAD1" device=""/>
 <part name="10F320" library="Microchip_By_element14_Batch_1" deviceset="PIC10F220T-I/OT" device="" value="PIC10F320T-I/OT"/>
@@
 <part name="JP4" library="SparkFun-Connectors" deviceset="M03" device="POLAR"/>
 <part name="GND3" library="supply1" deviceset="GND" device=""/>
-<part name="R4" library="SparkFun-Resistors" deviceset="RESISTOR" device="0805-RES" value="10K"/>
+<part name="R4" library="SparkFun-Resistors" deviceset="RESISTOR" device="0805-RES" value="1K"/>
 <part name="C3" library="SparkFun-Capacitors" deviceset="CAP" device="" value="0.1uF"/>
-<part name="R5" library="SparkFun-Resistors" deviceset="RESISTOR" device="0805-RES" value="10K"/>
-<part name="R6" library="SparkFun-Resistors" deviceset="RESISTOR" device="0805-RES" value="10K"/>
+<part name="R5" library="SparkFun-Resistors" deviceset="RESISTOR" device="0805-RES" value="5K6"/>
+<part name="R6" library="SparkFun-Resistors" deviceset="RESISTOR" device="0805-RES" value="4K7"/>
 <part name="GND4" library="supply1" deviceset="GND" device=""/>
 <part name="P+1" library="supply1" deviceset="+5V" device=""/>
@@
 <part name="Q4" library="SparkFun-DiscreteSemi" deviceset="TRANSISTOR_PNP" device="SMD" value="P-FET"/>
 <part name="GND10" library="supply1" deviceset="GND" device=""/>
-<part name="R9" library="SparkFun-Resistors" deviceset="RESISTOR" device="0805-RES" value="10K"/>
+<part name="R9" library="SparkFun-Resistors" deviceset="RESISTOR" device="0805-RES" value="4K7"/>
 <part name="Q5" library="SparkFun-DiscreteSemi" deviceset="TRANSISTOR_PNP" device="SMD" value="P-FET"/>
-<part name="R10" library="SparkFun-Resistors" deviceset="RESISTOR" device="0805-RES" value="10K"/>
+<part name="R10" library="SparkFun-Resistors" deviceset="RESISTOR" device="0805-RES" value="4K7"/>
 <part name="GND15" library="supply1" deviceset="GND" device=""/>
+<part name="Q1" library="SparkFun-DiscreteSemi" deviceset="TRANSISTOR_NPN" device="SOT23-3"/>
 </parts>
 <sheets>
@@
 <instance part="." gate="G$1" x="200.66" y="111.76" rot="R180"/>
 <instance part="C1" gate="G$1" x="25.4" y="78.74" rot="MR0"/>
-<instance part="Q1" gate="G$1" x="106.68" y="162.56" rot="MR0"/>
 <instance part="U$3" gate="G$1" x="160.02" y="180.34" rot="R180"/>
 <instance part="10F320" gate="A" x="83.82" y="35.56"/>
@@
 <instance part="R10" gate="G$1" x="40.64" y="139.7" rot="R90"/>
 <instance part="GND15" gate="1" x="40.64" y="114.3" rot="MR0"/>
+<instance part="Q1" gate="G$1" x="106.68" y="162.56" rot="MR0"/>
 </instances>
 <busses>
@@
 </segment>
 <segment>
-<pinref part="Q1" gate="G$1" pin="C"/>
 <pinref part="GND14" gate="1" pin="GND"/>
 <wire x1="104.14" y1="157.48" x2="104.14" y2="154.94" width="0.1524" layer="91"/>
@@
 <junction x="104.14" y="154.94"/>
 <pinref part="JP6" gate="G$1" pin="1"/>
+<pinref part="Q1" gate="G$1" pin="E"/>
 </segment>
 <segment>
@@
 <segment>
 <wire x1="99.06" y1="172.72" x2="104.14" y2="172.72" width="0.1524" layer="91"/>
-<pinref part="Q1" gate="G$1" pin="E"/>
 <wire x1="104.14" y1="172.72" x2="104.14" y2="167.64" width="0.1524" layer="91"/>
 <pinref part="JP6" gate="G$1" pin="2"/>
+<pinref part="Q1" gate="G$1" pin="C"/>
 </segment>
 </net>
@@
 <net name="N$8" class="0">
 <segment>
-<pinref part="Q1" gate="G$1" pin="B"/>
 <pinref part="R4" gate="G$1" pin="1"/>
 <wire x1="109.22" y1="162.56" x2="111.76" y2="162.56" width="0.1524" layer="91"/>
-</segment>
-</net>
+<pinref part="Q1" gate="G$1" pin="B"/>
+</segment>
+</net>

Commit message: Simplified, added DHT22
Parts:
- removed 10F320: PIC10F320T-I/OT, Microchip_By_element14_Batch_1:PIC10F220T-I/OT
- removed 3V3, JP5: (no value), SparkFun-Connectors:M01PTH
- removed JP4: (no value), SparkFun-Connectors:M03POLAR
- removed Q2, Q3: (no value), SparkFun-DiscreteSemi:TRANSISTOR_NPNSOT23-3
- removed Q4, Q5: P-FET, SparkFun-DiscreteSemi:TRANSISTOR_PNPSMD
- removed R10, R9: 4K7, SparkFun-Resistors:RESISTOR0805-RES
- removed R7, R8: 330, SparkFun-Resistors:RESISTOR0805-RES
- removed U$3: SMD-PAD1, CuriousTech:SMD-PAD1
- removed U$9: PIC-ICSP-MINI, SparkFun-Connectors:PIC-ICSP-MINI
- added U$4: USB-MINIB-5PIN, SparkFun-Connectors:USB-MINIB-5PIN
- JP1: value USB-MICROB -> (none); device SparkFun-Connectors:USB-MICROB -> SparkFun-Connectors:M04POLAR
- JP3: device SparkFun-Connectors:M03POLAR -> SparkFun-Connectors:M04POLAR
Connections:
- removed net ICSPDAT: 10F320.GP0/AN0/ICSPDAT, R4.2, U$9.PGD
- removed net N$12: Q2.C, Q5.B, R10.1
- removed net N$13: JP3.2, Q5.C
- removed net N$2: JP2.2, Q4.C
- removed net N$5: JP5.1, R7.2
- removed net N$6: Q3.C, Q4.B, R9.1
- net +5V: now also JP1.4, JP2.2, JP3.4, U$4.VBUS; no longer JP1.VBUS, JP4.2, Q4.E, Q5.E, R10.2, R9.2, U$3.P$1
- net 3V3: now also JP6.3; no longer 10F320.VDD, 3V3.1
- net ANA: no longer JP3.3
- net GND: now also JP1.1, U$4.GND, U$4.MTN1, U$4.MTN2, U$4.MTN3, U$4.MTN4; no longer 10F320.VSS, JP1.GND, JP4.1, Q2.E, Q3.E, R8.1, U$9.GND
- net ICSPCLK: no longer 10F320.GP1/AN1/ICSPCLK, U$9.PGC
- net IO0: no longer JP6.3
- net IO12: now also JP1.2; no longer JP4.3
- net IO13: now also JP1.3; no longer R7.1, R8.2
- net IO14: now also JP3.3; no longer Q2.B
- net IO15: now also R4.2; no longer 10F320.GP3/~MCLR/VPP, U$9.VPP
- net IO16: now also JP3.2; no longer Q3.B
- net IO2: no longer 10F320.GP2/T0CKI/FOSC4
Other:
- moved on the sheet: 3V3R, C3, C4
